File: Europe-flex.kicad_sch (KiCad schematic)
At the start: 399 parts, among them J1 Conn_01x04_Male/I2C, J10 Conn_01x06_Male, J100 Conn_01x02_Male, J101 Conn_01x02_Male, J102 Conn_01x02_Male, J103 Conn_01x02_Male, J104 Conn_01x01_Male, J105 Conn_01x02_Male, J106 Conn_01x02_Male, J107 Conn_01x02_Male, J108 Conn_01x02_Male, J109 Conn_01x02_Male, J11 Conn_01x02_Male, J110 Conn_01x01_Male, J111 Conn_01x02_Male, J112 Conn_01x02_Male, J113 Conn_01x02_Male, J114 Conn_01x02_Male, J115 Conn_01x02_Male, J116 Conn_01x01_Male, J117 Conn_01x01_Male, J118 Conn_01x01_Male, J119 Conn_01x01_Male, J12 Conn_01x02_Male, J120 Conn_01x01_Male, J121 Conn_01x01_Male, J122 Conn_01x01_Male, J123 Conn_01x01_Male, J124 Conn_01x01_Male, J125 Conn_01x01_Male, J126 Conn_01x01_Male, J127 Conn_01x01_Male, J128 Conn_01x01_Male, J129 Conn_01x01_Male, J13 Conn_01x02_Male, J130 Conn_01x01_Male, J131 Conn_01x01_Male, J132 Conn_01x01_Male, J133 Conn_01x01_Male, J134 Conn_01x01_Male, J135 Conn_01x01_Male, J136 Conn_01x01_Male, J137 Conn_01x01_Male, J138 Conn_01x01_Male, J139 Conn_01x01_Male, J14 Conn_01x02_Male, J140 Conn_01x01_Male, J141 Conn_01x01_Male, J142 Conn_01x01_Male, J143 Conn_01x01_Male, J144 Conn_01x01_Male, J145 Conn_01x01_Male, J146 Conn_01x01_Male, J147 Conn_01x01_Male, J148 Conn_01x01_Male, J149 Conn_01x01_Male, J15 Conn_01x01_Male, J150 Conn_01x01_Male, J151 Conn_01x01_Male, J152 Conn_01x01_Male, J153 Conn_01x01_Male, J16 Conn_01x02_Male, J17 Conn_01x02_Male, J18 Conn_01x02_Male, J19 Conn_01x02_Male, J2 Conn_01x04_Male, J20 Conn_01x02_Male, J21 Conn_01x01_Male, J22 Conn_01x02_Male, J23 Conn_01x02_Male, J24 Conn_01x02_Male, J25 Conn_01x02_Male, J26 Conn_01x01_Female, J27 Conn_01x01_Female, J28 Conn_01x01_Female, J29 Conn_01x01_Female, J3 Conn_01x06_Male, J30 Conn_01x01_Female, J31 Conn_01x01_Female, J32 Conn_01x01_Female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

Commit message: Add files via upload
Parts:
- added H3, H37, H38, H4: MountingHole_Pad, MountingHole:MountingHole_4.3mm_M4_DIN965_Pad, symbol Mechanical:MountingHole_Pad
Connections:
- net GNDL: now also H3.1, H4.1
- net GNDR: now also H21.1, H27.1, H37.1, H38.1
Other:
- moved on the sheet: H1, H10, H11, H12, H16, H17, H18, H19, H2, H20, H21, H22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

Commit message: Add files via upload
Parts:
- removed J101, J103, J105, J107, J109, J111, J113, J115, J12, J14, J16, J18, J20, J22, J24, J37, J38, J40, J42, J44, J46, J48, J50, J52, J54, J57, J59, J61, J64, J66, J69, J73, J75, J77, J79, J81, J82, J84, J87, J89, J9, J91, J93, J95, J97, J99: Conn_01x02_Male, Connector_PinHeader_2.54mm:PinHeader_1x02_P2.54mm_Vertical, symbol Connector:Conn_01x02_Male
- removed J123, J124, J125, J126, J127, J56, J67, J80: Conn_01x01_Male, Connector_PinHeader_2.54mm:PinHeader_1x01_P2.54mm_Vertical, symbol Connector:Conn_01x01_Male
- added J12, J16, J18, J20, J9: Conn_01x01_Male, Connector_PinHeader_2.54mm:PinHeader_1x01_P2.54mm_Vertical, symbol Connector:Conn_01x01_Male
- added J14, J22, J24, J37: Conn_01x03_Female, Connector_PinHeader_2.54mm:PinHeader_1x03_P2.54mm_Vertical, symbol Connector:Conn_01x03_Female
- J26, J27, J28, J29, J30, J31, J32, J33, J34, J35, J36, J4: footprint Connector_PinSocket_2.54mm:PinSocket_1x01_P2.54mm_Vertical -> Connector_PinHeader_2.54mm:PinHeader_1x01_P2.54mm_Vertical
- J45: footprint Connector_PinHeader_2.54mm:PinHeader_1x02_P2.54mm_Vertical -> Connector_PinHeader_2.54mm:PinHeader_1x01_P2.54mm_Vertical
Connections:
- net Arrow-Left: now also J5.1 (Pin_1); no longer J5.9 (Pin_9)
- net Arrow-Right: now also J8.1 (Pin_1); no longer J8.9 (Pin_9)
- net COL1: now also J5.9 (Pin_9); no longer J5.1 (Pin_1)
- net COL1R: now also J8.9 (Pin_9); no longer J8.1 (Pin_1)
- net COL1_L: now also D99.1 (K), J6.9 (Pin_9); no longer J6.1 (Pin_1)
- net COL2: now also J5.8 (Pin_8); no longer J5.2 (Pin_2)
- net COL2R: now also J8.8 (Pin_8); no longer J8.2 (Pin_2)
- net COL2_L: now also D95.1 (K), J6.8 (Pin_8); no longer J6.2 (Pin_2)
- net COL3: now also J5.7 (Pin_7); no longer J5.3 (Pin_3)
- net COL3R: now also J8.7 (Pin_7); no longer J8.3 (Pin_3)
- net COL3_L: now also D89.1 (K), J6.7 (Pin_7); no longer J6.3 (Pin_3)
- net COL4: now also J5.6 (Pin_6); no longer J5.4 (Pin_4)
- net COL4R: now also J8.6 (Pin_6); no longer J8.4 (Pin_4)
- net COL4_L: now also D82.1 (K), J6.6 (Pin_6); no longer J6.4 (Pin_4)
- net COL5_L: now also D75.1 (K)
- net COL6: now also J5.4 (Pin_4); no longer J5.6 (Pin_6)
- net COL6R: now also J8.4 (Pin_4); no longer J8.6 (Pin_6)
- net COL6_L: now also D71.1 (K), J6.4 (Pin_4); no longer D67.1 (K)
- net COL7: now also J5.3 (Pin_3); no longer J5.7 (Pin_7)
- net COL7R: now also J8.3 (Pin_3); no longer J8.7 (Pin_7)
- net COL8: now also J5.2 (Pin_2); no longer J5.8 (Pin_8)
- net COL8R: now also J8.2 (Pin_2); no longer J8.8 (Pin_8)
- net COL8_L: now also J14.2 (Pin_2), J18.1 (Pin_1)
- net COL9_L: now also J14.1 (Pin_1), J20.1 (Pin_1); no longer J116.1 (Pin_1)
- net at D1.1 (K): now also D2.1 (K), J112.1 (Pin_1), J112.2 (Pin_2)
- net at D7.1 (K): now also D8.1 (K), J106.1 (Pin_1), J106.2 (Pin_2)
- net at D3.1 (K): now also D4.1 (K), J114.1 (Pin_1), J114.2 (Pin_2)
- net at D9.1 (K): now also D10.1 (K), J108.1 (Pin_1), J108.2 (Pin_2)
- net at D5.1 (K): now also D6.1 (K), J110.1 (Pin_1), J7.9 (Pin_9)
- net at D11.1 (K): now also D12.1 (K), J104.1 (Pin_1), J7.8 (Pin_8)
- net at D18.1 (K), J7.7 (Pin_7), J98.1 (Pin_1): now also D16.1 (K)
- net at D17.1 (K), J102.1 (Pin_1), J102.2 (Pin_2): now also D15.1 (K)
- net at D14.1 (K), J100.1 (Pin_1), J100.2 (Pin_2): now also D13.1 (K)
- net at D19.1 (K): now also D20.1 (K), J94.1 (Pin_1), J94.2 (Pin_2)
- net at D22.1 (K), J96.1 (Pin_1), J96.2 (Pin_2): now also D21.1 (K)
- net at D23.1 (K): now also D24.1 (K), J7.6 (Pin_6), J92.1 (Pin_1)
- net at D30.1 (K), J7.5 (Pin_5), J86.1 (Pin_1): now also D29.1 (K)
- net at D28.1 (K), J90.1 (Pin_1), J90.2 (Pin_2): now also D26.1 (K)
- net at D27.1 (K), J88.1 (Pin_1), J88.2 (Pin_2): now also D25.1 (K)
- net at D35.1 (K): now also J128.1 (Pin_1)
- net at D34.1 (K), J85.1 (Pin_1), J85.2 (Pin_2): now also D33.1 (K)
- net at D32.1 (K), J83.1 (Pin_1), J83.2 (Pin_2): now also D31.1 (K)
- net at D39.1 (K): now also J7.4 (Pin_4), J74.1 (Pin_1)
- net at D41.1 (K), J78.1 (Pin_1), J78.2 (Pin_2): now also D40.1 (K)
- net at D38.1 (K), J76.1 (Pin_1), J76.2 (Pin_2): now also D37.1 (K)
- net at D45.1 (K): now also J70.1 (Pin_1)
- net at D46.1 (K): now also J68.1 (Pin_1)
- net at D36.1 (K): now also J37.3 (Pin_3)
- net at D44.1 (K): now also J37.2 (Pin_2); no longer J70.1 (Pin_1)
- net at D47.1 (K): now also J37.1 (Pin_1); no longer J68.1 (Pin_1)
- net at J7.3 (Pin_3): now also J24.3 (Pin_3); no longer J74.1 (Pin_1)
- net at D77.1 (K): now also D74.1 (K), J47.1 (Pin_1), J47.2 (Pin_2)
- net at D92.1 (K), J17.1 (Pin_1), J17.2 (Pin_2): now also D96.1 (K)
- net at D78.1 (K): now also D73.1 (K), J45.1 (Pin_1), J45.2 (Pin_2)
- net at D100.1 (K), J11.1 (Pin_1), J11.2 (Pin_2): now also D102.1 (K)
- net at D87.1 (K), J23.1 (Pin_1), J23.2 (Pin_2): now also D90.1 (K)
- net at D84.1 (K): now also D79.1 (K), J39.1 (Pin_1), J39.2 (Pin_2)
- net at D68.1 (K), J51.1 (Pin_1), J51.2 (Pin_2): now also D72.1 (K)
- net at D65.1 (K): now also J12.1 (Pin_1)
- net at D88.1 (K): now also D85.1 (K), J25.1 (Pin_1), J25.2 (Pin_2)
- net at D80.1 (K): now also D81.1 (K), J41.1 (Pin_1), J41.2 (Pin_2)
- net at D62.1 (K): now also D63.1 (K), J60.1 (Pin_1), J60.2 (Pin_2)
- net at D66.1 (K): now also D64.1 (K), J58.1 (Pin_1), J58.2 (Pin_2)
- net at D93.1 (K): now also D94.1 (K), J19.1 (Pin_1), J19.2 (Pin_2)
- net at D101.1 (K): now also D98.1 (K), J13.1 (Pin_1), J13.2 (Pin_2)
- net at J7.1 (Pin_1): now also J24.1 (Pin_1)
- net at J7.2 (Pin_2): now also J24.2 (Pin_2)
- net at D69.1 (K): now also D70.1 (K), J53.1 (Pin_1), J53.2 (Pin_2)
- net at D58.1 (K): now also J16.1 (Pin_1)
- net at D57.1 (K): now also J116.1 (Pin_1)
- new net: D67.1 (K), J14.3 (Pin_3), J9.1 (Pin_1)
- new net: J22.1 (Pin_1), J6.1 (Pin_1)
- new net: J22.2 (Pin_2), J6.2 (Pin_2)
- new net: J22.3 (Pin_3), J6.3 (Pin_3)
Other:
- moved on the sheet: D67, J104, J110, J116, J121, J128, J15, J21, J43, J49, J5, J55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

Commit message: Add files via upload
Connections:
- net COL1_L: now also D100.1 (K), D101.1 (K), D102.1 (K), D98.1 (K), J11.1 (Pin_1), J11.2 (Pin_2), J13.1 (Pin_1), J13.2 (Pin_2)
- net COL2_L: now also D92.1 (K), D93.1 (K), D94.1 (K), D96.1 (K), J17.1 (Pin_1), J17.2 (Pin_2), J19.1 (Pin_1), J19.2 (Pin_2)
- net COL3_L: now also D85.1 (K), D87.1 (K), D88.1 (K), D90.1 (K), J23.1 (Pin_1), J23.2 (Pin_2), J25.1 (Pin_1), J25.2 (Pin_2)
- net COL4_L: now also D79.1 (K), D80.1 (K), D81.1 (K), D84.1 (K), J39.1 (Pin_1), J39.2 (Pin_2), J41.1 (Pin_1), J41.2 (Pin_2)
- net COL5_L: now also D73.1 (K), D74.1 (K), D77.1 (K), D78.1 (K), J45.1 (Pin_1), J45.2 (Pin_2), J47.1 (Pin_1), J47.2 (Pin_2)
- net COL6_L: now also D68.1 (K), D69.1 (K), D70.1 (K), D72.1 (K), J51.1 (Pin_1), J51.2 (Pin_2), J53.1 (Pin_1), J53.2 (Pin_2)
- net COL8_L: now also D59.1 (K), D60.1 (K), J62.1 (Pin_1), J62.2 (Pin_2), J63.1 (Pin_1), J63.2 (Pin_2)
- net COL9_L: now also D57.1 (K), J116.1 (Pin_1)
- net COL7_L: now reaches D67.1 (K), J14.3 (Pin_3), J9.1 (Pin_1)
- net COL7_L: now also D58.1 (K), D62.1 (K), D63.1 (K), D64.1 (K), D65.1 (K), D66.1 (K), J12.1 (Pin_1), J16.1 (Pin_1), J58.1 (Pin_1), J58.2 (Pin_2), J60.1 (Pin_1), J60.2 (Pin_2)
Other:
- note added: "Right and left sides separated by blue lines. Both sides are mirrored as much as possible."
- note removed: "Right and left sides separated by blue lines."
Changed lines of the file:
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@@
     (effects (font (size 1.27 1.27)) (justify left bottom))
   )
-  (text "Right and left sides separated by blue lines." (at 723.9 556.26 0)
+  (text "Right and left sides separated by blue lines.\nBoth sides are mirrored as much as possible."
+    (at 723.9 556.26 0)
     (effects (font (size 1.27 1.27)) (justify left bottom))
   )
@@
     (effects (font (size 1.27 1.27)) (justify left bottom))
   )
+  (label "COL4_L" (at 247.65 240.03 0)
+    (effects (font (size 1.27 1.27)) (justify left bottom))
+  )
+  (label "COL3_L" (at 222.25 238.76 0)
+    (effects (font (size 1.27 1.27)) (justify left bottom))
+  )
   (label "COL9_L" (at 378.46 344.17 0)
     (effects (font (size 1.27 1.27)) (justify left bottom))
@@
     (effects (font (size 1.27 1.27)) (justify left bottom))
   )
+  (label "COL4_L" (at 247.65 123.19 0)
+    (effects (font (size 1.27 1.27)) (justify left bottom))
+  )
+  (label "COL7_L" (at 351.79 289.56 0)
+    (effects (font (size 1.27 1.27)) (justify left bottom))
+  )
   (label "ROW3_L" (at 162.56 156.21 0)
+    (effects (font (size 1.27 1.27)) (justify left bottom))
+  )
+  (label "COL7_L" (at 317.5 237.49 0)
+    (effects (font (size 1.27 1.27)) (justify left bottom))
+  )
+  (label "COL5_L" (at 270.51 119.38 0)
+    (effects (font (size 1.27 1.27)) (justify left bottom))
+  )
+  (label "COL7_L" (at 321.31 344.17 0)
+    (effects (font (size 1.27 1.27)) (justify left bottom))
+  )
+  (label "COL7_L" (at 317.5 118.11 0)
     (effects (font (size 1.27 1.27)) (justify left bottom))
   )
@@
     (effects (font (size 1.27 1.27)) (justify left bottom))
   )
+  (label "COL5_L" (at 270.51 236.22 0)
+    (effects (font (size 1.27 1.27)) (justify left bottom))
+  )
   (label "ROW1_L" (at 162.56 40.64 0)
+    (effects (font (size 1.27 1.27)) (justify left bottom))
+  )
+  (label "COL8_L" (at 351.79 179.07 0)
+    (effects (font (size 1.27 1.27)) (justify left bottom))
+  )
+  (label "COL1_L" (at 173.99 233.68 0)
     (effects (font (size 1.27 1.27)) (justify left bottom))
   )
@@
     (effects (font (size 1.27 1.27)) (justify left bottom))
   )
+  (label "COL1_L" (at 173.99 121.92 0)
+    (effects (font (size 1.27 1.27)) (justify left bottom))
+  )
+  (label "COL2_L" (at 196.85 236.22 0)
+    (effects (font (size 1.27 1.27)) (justify left bottom))
+  )
   (label "ROW6_L" (at 163.83 320.04 0)
+    (effects (font (size 1.27 1.27)) (justify left bottom))
+  )
+  (label "COL6_L" (at 293.37 121.92 0)
     (effects (font (size 1.27 1.27)) (justify left bottom))
   )
@@
     (effects (font (size 1.27 1.27)) (justify left bottom))
   )
+  (label "COL8_L" (at 351.79 118.11 0)
+    (effects (font (size 1.27 1.27)) (justify left bottom))
+  )
   (label "COL8_L" (at 351.79 339.09 0)
     (effects (font (size 1.27 1.27)) (justify left bottom))
   )
+  (label "COL6_L" (at 293.37 237.49 0)
+    (effects (font (size 1.27 1.27)) (justify left bottom))
+  )
   (label "GNDL" (at 347.98 422.91 0)
+    (effects (font (size 1.27 1.27)) (justify left bottom))
+  )
+  (label "COL7_L" (at 317.5 290.83 0)
     (effects (font (size 1.27 1.27)) (justify left bottom))
   )
@@
     (effects (font (size 1.27 1.27)) (justify left bottom))
   )
+  (label "COL9_L" (at 378.46 289.56 0)
+    (effects (font (size 1.27 1.27)) (justify left bottom))
+  )
   (label "COL2_L" (at 196.85 344.17 0)
     (effects (font (size 1.27 1.27)) (justify left bottom))
   )
+  (label "COL3_L" (at 222.25 120.65 0)
+    (effects (font (size 1.27 1.27)) (justify left bottom))
+  )
+  (label "COL2_L" (at 196.85 124.46 0)
+    (effects (font (size 1.27 1.27)) (justify left bottom))
+  )

Commit message: Add files via upload
Connections:
- net COL7_L: no longer D62.1 (K), D63.1 (K), D64.1 (K), D66.1 (K), D67.1 (K), J14.3 (Pin_3), J58.1 (Pin_1), J58.2 (Pin_2), J60.1 (Pin_1), J60.2 (Pin_2), J9.1 (Pin_1)
- net COL8_L: no longer D60.1 (K), D61.1 (K), J14.2 (Pin_2), J18.1 (Pin_1), J62.1 (Pin_1), J62.2 (Pin_2)
- net COL9_L: no longer D56.1 (K), J14.1 (Pin_1), J20.1 (Pin_1)
- net GNDL: now also U2.42 (GND)
- net GNDR: now also U1.42 (GND)
- removed net COL1_L: D100.1 (K), D101.1 (K), D102.1 (K), D97.1 (K), D98.1 (K), D99.1 (K), J11.1 (Pin_1), J11.2 (Pin_2), J13.1 (Pin_1), J13.2 (Pin_2), J15.1 (Pin_1), J6.9 (Pin_9)
- removed net COL2_L: D91.1 (K), D92.1 (K), D93.1 (K), D94.1 (K), D95.1 (K), D96.1 (K), J17.1 (Pin_1), J17.2 (Pin_2), J19.1 (Pin_1), J19.2 (Pin_2), J21.1 (Pin_1), J6.8 (Pin_8)
- removed net COL3_L: D85.1 (K), D86.1 (K), D87.1 (K), D88.1 (K), D89.1 (K), D90.1 (K), J23.1 (Pin_1), J23.2 (Pin_2), J25.1 (Pin_1), J25.2 (Pin_2), J43.1 (Pin_1), J6.7 (Pin_7)
- removed net COL4_L: D79.1 (K), D80.1 (K), D81.1 (K), D82.1 (K), D83.1 (K), D84.1 (K), J39.1 (Pin_1), J39.2 (Pin_2), J41.1 (Pin_1), J41.2 (Pin_2), J49.1 (Pin_1), J6.6 (Pin_6)
- removed net COL5_L: D73.1 (K), D74.1 (K), D75.1 (K), D76.1 (K), D77.1 (K), D78.1 (K), J45.1 (Pin_1), J45.2 (Pin_2), J47.1 (Pin_1), J47.2 (Pin_2), J55.1 (Pin_1), J6.5 (Pin_5)
- removed net COL6_L: D68.1 (K), D69.1 (K), D70.1 (K), D71.1 (K), D72.1 (K), J51.1 (Pin_1), J51.2 (Pin_2), J53.1 (Pin_1), J53.2 (Pin_2), J6.4 (Pin_4), J65.1 (Pin_1)
- new net: D74.1 (K), D77.1 (K), J47.1 (Pin_1), J47.2 (Pin_2)
- new net: D92.1 (K), D96.1 (K), J17.1 (Pin_1), J17.2 (Pin_2)
- new net: D56.1 (K), J14.1 (Pin_1), J20.1 (Pin_1)
- new net: D61.1 (K), J14.2 (Pin_2), J18.1 (Pin_1)
- new net: D67.1 (K), J14.3 (Pin_3), J9.1 (Pin_1)
- new net: D71.1 (K), J6.4 (Pin_4), J65.1 (Pin_1)
- new net: D100.1 (K), D102.1 (K), J11.1 (Pin_1), J11.2 (Pin_2)
- new net: D87.1 (K), D90.1 (K), J23.1 (Pin_1), J23.2 (Pin_2)
- new net: D82.1 (K), D83.1 (K), J49.1 (Pin_1), J6.6 (Pin_6)
- new net: D86.1 (K), D89.1 (K), J43.1 (Pin_1), J6.7 (Pin_7)
- new net: D79.1 (K), D84.1 (K), J39.1 (Pin_1), J39.2 (Pin_2)
- new net: D68.1 (K), D72.1 (K), J51.1 (Pin_1), J51.2 (Pin_2)
- new net: D73.1 (K), D78.1 (K), J45.1 (Pin_1), J45.2 (Pin_2)
- new net: D85.1 (K), D88.1 (K), J25.1 (Pin_1), J25.2 (Pin_2)
- new net: D80.1 (K), D81.1 (K), J41.1 (Pin_1), J41.2 (Pin_2)
- new net: D97.1 (K), D99.1 (K), J15.1 (Pin_1), J6.9 (Pin_9)
- new net: D91.1 (K), D95.1 (K), J21.1 (Pin_1), J6.8 (Pin_8)
- new net: D62.1 (K), D63.1 (K), J60.1 (Pin_1), J60.2 (Pin_2)
- new net: D64.1 (K), D66.1 (K), J58.1 (Pin_1), J58.2 (Pin_2)
- new net: D93.1 (K), D94.1 (K), J19.1 (Pin_1), J19.2 (Pin_2)
- new net: D101.1 (K), D98.1 (K), J13.1 (Pin_1), J13.2 (Pin_2)
- new net: D69.1 (K), D70.1 (K), J53.1 (Pin_1), J53.2 (Pin_2)
- new net: D75.1 (K), D76.1 (K), J55.1 (Pin_1), J6.5 (Pin_5)
- new net: D60.1 (K), J62.1 (Pin_1), J62.2 (Pin_2)
- no-connect marks 23 -> 21
Changed lines of the file:
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@@
   (no_connect (at 345.44 410.21))
   (no_connect (at 325.12 455.93))
-  (no_connect (at 327.66 455.93))
   (no_connect (at 518.16 419.1))
   (no_connect (at 518.16 424.18))
@@
   (no_connect (at 345.44 412.75))
   (no_connect (at 497.84 464.82))
-  (no_connect (at 500.38 464.82))
   (no_connect (at 518.16 444.5))
   (no_connect (at 345.44 415.29))
@@
     (stroke (width 0) (type default) (color 0 0 0 0))
   )
+  (wire (pts (xy 327.66 455.93) (xy 327.66 458.47))
+    (stroke (width 0) (type default) (color 0 0 0 0))
+  )
   (wire (pts (xy 247.65 288.29) (xy 247.65 298.45))
     (stroke (width 0) (type default) (color 0 0 0 0))
@@
     (stroke (width 0) (type default) (color 0 0 0 0))
   )
+  (wire (pts (xy 500.38 464.82) (xy 500.38 468.63))
+    (stroke (width 0) (type default) (color 0 0 0 0))
+  )
   (polyline (pts (xy 12.7 15.24) (xy 12.7 579.12))
     (stroke (width 0) (type default) (color 0 0 0 0))
@@
     (effects (font (size 1.27 1.27)) (justify left bottom))
   )
-  (label "COL3_L" (at 222.25 341.63 0)
-    (effects (font (size 1.27 1.27)) (justify left bottom))
-  )
-  (label "COL4_L" (at 247.65 240.03 0)
-    (effects (font (size 1.27 1.27)) (justify left bottom))
-  )
-  (label "COL3_L" (at 222.25 238.76 0)
-    (effects (font (size 1.27 1.27)) (justify left bottom))
-  )
-  (label "COL9_L" (at 378.46 344.17 0)
-    (effects (font (size 1.27 1.27)) (justify left bottom))
-  )
-  (label "COL6_L" (at 293.37 340.36 0)
-    (effects (font (size 1.27 1.27)) (justify left bottom))
-  )
-  (label "COL4_L" (at 247.65 123.19 0)
-    (effects (font (size 1.27 1.27)) (justify left bottom))
-  )
   (label "COL7_L" (at 351.79 289.56 0)
     (effects (font (size 1.27 1.27)) (justify left bottom))
@@
     (effects (font (size 1.27 1.27)) (justify left bottom))
   )
-  (label "COL7_L" (at 317.5 237.49 0)
-    (effects (font (size 1.27 1.27)) (justify left bottom))
-  )
-  (label "COL5_L" (at 270.51 119.38 0)
-    (effects (font (size 1.27 1.27)) (justify left bottom))
-  )
-  (label "COL7_L" (at 321.31 344.17 0)
-    (effects (font (size 1.27 1.27)) (justify left bottom))
-  )
-  (label "COL7_L" (at 317.5 118.11 0)
-    (effects (font (size 1.27 1.27)) (justify left bottom))
-  )
   (label "ROW2_L" (at 166.37 93.98 0)
     (effects (font (size 1.27 1.27)) (justify left bottom))
   )
-  (label "COL4_L" (at 247.65 340.36 0)
-    (effects (font (size 1.27 1.27)) (justify left bottom))
-  )
-  (label "COL5_L" (at 270.51 236.22 0)
-    (effects (font (size 1.27 1.27)) (justify left bottom))
-  )
   (label "ROW1_L" (at 162.56 40.64 0)
     (effects (font (size 1.27 1.27)) (justify left bottom))
@@
     (effects (font (size 1.27 1.27)) (justify left bottom))
   )
-  (label "COL1_L" (at 173.99 233.68 0)
-    (effects (font (size 1.27 1.27)) (justify left bottom))
-  )
-  (label "COL5_L" (at 270.51 339.09 0)
-    (effects (font (size 1.27 1.27)) (justify left bottom))
-  )
-  (label "COL1_L" (at 173.99 121.92 0)
-    (effects (font (size 1.27 1.27)) (justify left bottom))
-  )
-  (label "COL2_L" (at 196.85 236.22 0)
-    (effects (font (size 1.27 1.27)) (justify left bottom))
-  )
   (label "ROW6_L" (at 163.83 320.04 0)
     (effects (font (size 1.27 1.27)) (justify left bottom))
   )
-  (label "COL6_L" (at 293.37 121.92 0)
-    (effects (font (size 1.27 1.27)) (justify left bottom))
-  )
-  (label "COL1_L" (at 173.99 350.52 0)
-    (effects (font (size 1.27 1.27)) (justify left bottom))
-  )
-  (label "COL8_L" (at 351.79 118.11 0)
-    (effects (font (size 1.27 1.27)) (justify left bottom))
-  )
-  (label "COL8_L" (at 351.79 339.09 0)
-    (effects (font (size 1.27 1.27)) (justify left bottom))
-  )
-  (label "COL6_L" (at 293.37 237.49 0)
-    (effects (font (size 1.27 1.27)) (justify left bottom))
-  )
   (label "GNDL" (at 347.98 422.91 0)
     (effects (font (size 1.27 1.27)) (justify left bottom))
@@
     (effects (font (size 1.27 1.27)) (justify left bottom))
   )
-  (label "COL2_L" (at 196.85 344.17 0)
-    (effects (font (size 1.27 1.27)) (justify left bottom))
-  )
-  (label "COL3_L" (at 222.25 120.65 0)
-    (effects (font (size 1.27 1.27)) (justify left bottom))
-  )
-  (label "COL2_L" (at 196.85 124.46 0)
-    (effects (font (size 1.27 1.27)) (justify left bottom))
-  )
   (global_label "ROW4R" (shape bidirectional) (at 471.17 434.34 180) (fields_autoplaced)
     (effects (font (size 1.27 1.27)) (justify right))
@@
     )
   )
+  (global_label "GNDL" (shape bidirectional) (at 327.66 458.47 0) (fields_autoplaced)
+    (effects (font (size 1.27 1.27)) (justify left))
+    (property "Intersheet References" "${INTERSHEET_REFS}" (id 0) (at 334.9717 458.5494 0)
+      (effects (font (size 1.27 1.27)) (justify left) hide)
+    )
+  )
   (global_label "ROW3" (shape input) (at 347.98 478.79 0) (fields_autoplaced)
     (effects (font (size 1.27 1.27)) (justify left))
@@
       (effects (font (size 1.27 1.27)) (justify left) hide)
     )
+  )
+  (global_label "GNDR" (shape input) (at 500.38 468.63 0) (fields_autoplaced)
+    (effects (font (size 1.27 1.27)) (justify left))
+    (property "Intersheet References" "${INTERSHEET_REFS}" (id 0) (at 507.8447 468.5506 0)
+      (effects (font (size 1.27 1.27)) (justify left) hide)
+    )

Commit message: Add files via upload
Parts:
- removed J1: Conn_01x04_Male/I2C, switch:CUI_SJ-43514, symbol Connector:Conn_01x04_Male
- removed J2: Conn_01x04_Male, switch:CUI_SJ-43514, symbol Connector:Conn_01x04_Male
- added J104, J93: SJ-435107, sj-conn:CUI_SJ-435107, symbol SJ:SJ-435107
- renumbered D7 to D1, D66 to D10, D54 to D100, D53 to D101, D52 to D102, D25 to D11, D19 to D12, D84 to D13, D78 to D14, D100 to D15, D92 to D16, D60 to D17, D42 to D18, D8 to D19, D1 to D2, D2 to D20, D87 to D21, D79 to D22, D73 to D23, D68 to D24, D64 to D25, D38 to D26, D32 to D27, D27 to D28, D20 to D29, D37 to D3, D14 to D30, D101 to D31, D93 to D32, D59 to D33, D69 to D34, D62 to D35, D88 to D36, D80 to D37, D77 to D38, D43 to D39, D31 to D4, D9 to D40, D3 to D41, D40 to D42, D33 to D43, D15 to D44, D26 to D45, D21 to D46, D98 to D47, D94 to D48, D74 to D49, D13 to D5, D70 to D50, D63 to D51, D85 to D52, D81 to D53, D10 to D54, D4 to D55, D41 to D56, D34 to D57, D28 to D58, D22 to D59, D102 to D6, D17 to D60, D99 to D61, D95 to D62, D58 to D63, D57 to D64, D89 to D65, D82 to D66, D75 to D67, D71 to D68, D65 to D69, D96 to D7, D46 to D70, D45 to D71, D11 to D72, D5 to D73, D35 to D74, D29 to D75, D23 to D76, D16 to D77, D39 to D78, D97 to D79, D90 to D8, D91 to D80, D67 to D81, D61 to D82, D56 to D83, D86 to D84, D76 to D85, D83 to D86, D47 to D87, D44 to D88, D36 to D89, D72 to D9, D12 to D90, D6 to D91, D18 to D92, D30 to D93, D24 to D94, D48 to D95, D49 to D96, D50 to D97, D51 to D98, D55 to D99, H21 to H1, H28 to H10, H2 to H11, H16 to H12, H23 to H13, H29 to H14, H8 to H15, H17 to H16, H24 to H17, H30 to H18, H9 to H19, H27 to H2, H18 to H20, H25 to H21, H31 to H22, H10 to H23, H19 to H24, H35 to H25, H36 to H26, H33 to H27, H34 to H28, H3 to H29, H1 to H3, H38 to H30, H4 to H31, H13 to H32, H37 to H33, H14 to H34, H5 to H35, H15 to H36, H6 to H37, H7 to H38, H12 to H4, H26 to H5, H32 to H6, H11 to H7, H20 to H8, H22 to H9, J33 to J1, J23 to J10, J132 to J100, J130 to J101, J136 to J102, J138 to J103, J143 to J105, J144 to J106, J133 to J107, J134 to J108, J76 to J11, J83 to J12, J88 to J13, J94 to J14, J100 to J15, J11 to J16, J62 to J17, J51 to J18, J39 to J19, J26 to J2, J17 to J20, J35 to J21, J28 to J22, J63 to J23, J72 to J24, J34 to J25, J29 to J26, J13 to J27, J47 to J28, J25 to J29, J36 to J3, J19 to J30, J41 to J31, J53 to J32, J60 to J33, J119 to J34, J118 to J35, J108 to J36, J114 to J37, J32 to J38, J78 to J39, J27 to J4, J85 to J40, J90 to J41, J96 to J42, J102 to J43, J120 to J44, J30 to J45, J15 to J46, J21 to J47, J43 to J48, J16 to J49, J71 to J5, J116 to J50, J49 to J51, J65 to J52, J12 to J53, J55 to J54, J117 to J55, J70 to J56, J104 to J57, J110 to J58, J4 to J59, J106 to J6, J92 to J60, J98 to J61, J68 to J62, J86 to J63, J128 to J64, J74 to J65, J18 to J66, J20 to J67, J121 to J68, J9 to J69, J112 to J7, J31 to J70, J14 to J71, J22 to J72, J37 to J73, J6 to J74, J24 to J75, J7 to J76, J5 to J77, J8 to J78, J149 to J79, J45 to J8, J122 to J80, J150 to J81, J151 to J82, J153 to J83, J152 to J84, J3 to J85, J10 to J86, J141 to J87, J145 to J88, J147 to J89, J58 to J9, J139 to J90, J129 to J91, J131 to J92, J135 to J94, J137 to J95, J146 to J96, J148 to J97, J140 to J98, J142 to J99, R3 to R1, R8 to R11, R7 to R12, R5 to R2, R1 to R3, R2 to R4, R4 to R5, R9 to R7, R11 to R8, R12 to R9, SW37 to SW1, SW84 to SW10, SW78 to SW11, SW72 to SW12, SW66 to SW13, SW60 to SW14, SW93 to SW15, SW87 to SW16, SW81 to SW17, SW75 to SW18, SW69 to SW19, SW31 to SW2, SW62 to SW20, SW57 to SW21, SW52 to SW22, SW42 to SW23, SW38 to SW24, SW32 to SW25, SW20 to SW27, SW14 to SW28, SW8 to SW29, SW25 to SW3, SW2 to SW30, SW94 to SW31, SW88 to SW32, SW82 to SW33, SW76 to SW34, SW70 to SW35, SW63 to SW36, SW58 to SW37, SW53 to SW38, SW43 to SW39, SW19 to SW4, SW39 to SW40, SW33 to SW41, SW27 to SW42, SW21 to SW43, SW15 to SW44, SW9 to SW45, SW3 to SW46, SW91 to SW47, SW85 to SW48, SW79 to SW49, SW13 to SW5, SW73 to SW50, SW67 to SW51, SW61 to SW52, SW56 to SW53, SW41 to SW54, SW36 to SW55, SW29 to SW56, SW23 to SW57, SW17 to SW58, SW11 to SW59, SW7 to SW6, SW5 to SW60, SW95 to SW61, SW89 to SW62, SW83 to SW63, SW77 to SW64, SW71 to SW65, SW64 to SW66, SW59 to SW67, SW54 to SW68, SW51 to SW69, SW1 to SW7, SW46 to SW70, SW44 to SW71, SW40 to SW72, SW34 to SW73, SW28 to SW74, SW22 to SW75, SW16 to SW76, SW10 to SW77, SW4 to SW78, SW92 to SW79, SW96 to SW8, SW86 to SW80, SW80 to SW81, SW74 to SW82, SW68 to SW83, SW65 to SW84, SW55 to SW85, SW50 to SW86, SW47 to SW87, SW45 to SW88, SW35 to SW89, SW90 to SW9, SW30 to SW90, SW24 to SW91, SW18 to SW92, SW12 to SW93, SW6 to SW94, SW49 to SW95, SW48 to SW96, U2 to U1, U1 to U2
Connections:
- net GNDL: now also J104.1
- net GNDR: now also J93.1
- net SCL I2C0: now also J104.2
- net SDA I2C0: now also J104.4
- net VCCL: now also J104.3
- net VCCR: now also J93.3
- net sclR: now also J93.2
- net sdaR: now also J93.4
